File: Electrical/IDP/Work In Progress.brd (EAGLE design)
At the start: 106.7 x 53.3 mm, 63 parts, among them IC1 NE555N, IC2 7414N, IC3 LM348P, IC4 7414N, IC5 LM348P, M1 IDP_PROTOBOARD_LARGE_LARGE, M2 IDP_PROTOBOARD_LARGE_LARGE, Q1 ARDUINOR3-NOIOREF-NOTEXT, U1 SN74HC02N, U2 HC-SR04, U6 HC-SR04

Commit message: Completed Line Follower routing
Parts:
- removed IC4: 7414N, IDP_library:DIL14
- removed IC5: LM348P, IDP_library:DIL14
- C4, C5: device IDP_library:C075-032X103 -> IDP_library:C025-024X044
- R1, R10, R11, R12, R13, R14, R15, R16, R17, R18, R19, R2, R20, R21, R22, R23, R24, R25, R26, R27, R28, R29, R3, R30, R4, R5, R6, R7, R8, R9: device IDP_library:0204/7 -> IDP_library:0204V
- U2, U6: value HC-SR04 -> HC-SR04CON; device IDP_library:XCVR_HC-SR04 -> IDP_library:22-23-2041
- moved M2 380.1 mm to (-81.3, 55.9)
- moved C5 356.2 mm to (-120.7, 179.1)
- moved U6 319.5 mm to (-130.8, 115.6)
- moved R16 287.0 mm to (-100.3, 73.7), turned to 180 degrees
- moved LED8 279.4 mm to (-153.7, -38.1)
- moved R29 279.4 mm to (-156.2, -59.7)
- moved R30 279.4 mm to (-146.1, -59.7)
- moved LED5 278.7 mm to (-99.1, 64.8), turned to 270 degrees
- moved U3 274.8 mm to (-114.3, 95.2), turned to 270 degrees
- moved LED3 270.9 mm to (-94.0, 95.2), turned to 90 degrees
- moved VR1 269.4 mm to (-152.4, -29.2)
- moved R25 269.2 mm to (-156.2, -54.6)
- moved R26 269.2 mm to (-146.1, -54.6)
- moved R27 269.2 mm to (-135.9, -54.6)
- moved R6 263.9 mm to (-102.9, 88.9), turned to 180 degrees
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Connections:
- net D0: no longer IC2.10, IC2.12, IC2.2, IC2.8, R10.2, R13.2, R16.2, R7.2
- net D1: now also IC2.12, R7.2
- net D2: now also IC2.10, R10.2
- net D3: now also IC2.8, R13.2
- net D4: now also IC2.2, R16.2
- net GND: no longer IC4.7
- net N$16: now also IC2.3; no longer IC4.5
- net N$22: now also IC2.4; no longer IC4.6
- net N$24: now also IC2.5, IC3.7; no longer IC4.3, IC5.1
- net N$25: now also IC3.6; no longer IC5.2
- net N$26: now also IC3.5; no longer IC5.3
- net N$30: now also IC2.6; no longer IC4.4
- net V+: no longer IC5.4
- net V-: no longer IC5.11
- net VCC: no longer IC4.14
Routing:
- net N$10: track 7.62 -> 54.0 mm, vias 0 -> 2
- net GND: track 123.5 -> 157.6 mm, vias 0 -> 14
- net N$5: track 0.00 -> 17.8 mm, vias 0 -> 3
- net N$7: track 23.9 -> 39.6 mm, vias 0 -> 2
- net N$12: track 10.2 -> 23.0 mm, vias 0 -> 2
- net N$4: track 14.0 -> 2.54 mm
- net N$2: track 0.00 -> 11.2 mm, vias 0 -> 2
- net +5V: track 2.54 -> 11.2 mm
- net N$14: track 0.00 -> 7.62 mm
- net D4: track 0.00 -> 5.08 mm
- net N$6: track 7.62 -> 12.0 mm, vias 0 -> 2
- net D3: track 0.00 -> 3.81 mm
- net D0: track 3.81 -> 0.00 mm
- net N$9: track 7.62 -> 11.4 mm, vias 0 -> 2
- net N$13: track 22.4 -> 19.7 mm, vias 0 -> 2
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Other:
- board size 106.7 x 53.3 mm -> 160 x 100 mm
- board text added: "x"
