File: Electrical/IDP/Work In Progress.sch (EAGLE design)
At the start: 63 parts, among them IC1 NE555N, IC2 7414N, IC3 LM348P, IC4 7414N, IC5 LM348P, M1 IDP_PROTOBOARD_LARGE_LARGE, M2 IDP_PROTOBOARD_LARGE_LARGE, Q1 ARDUINOR3-NOIOREF-NOTEXT, U1 SN74HC02N, U2 HC-SR04, U6 HC-SR04

Commit message: Completed Line Follower routing
Parts:
- removed IC4: 7414N, IDP_library:7414N
- removed IC5: LM348P, IDP_library:LM348P
- C4, C5: device IDP_library:C-EU075-032X103 -> IDP_library:C-EU025-024X044
- R1, R10, R11, R12, R13, R14, R15, R16, R17, R18, R19, R2, R20, R21, R22, R23, R24, R25, R26, R27, R28, R29, R3, R30, R4, R5, R6, R7, R8, R9: device IDP_library:R-EU_0204/7 -> IDP_library:R-EU_0204/2V
- U2, U6: value HC-SR04 -> HC-SR04CON; device IDP_library:HC-SR04 -> IDP_library:HC-SR04CON
Connections:
- net D0: no longer IC2A.O, IC2B.O, IC2C.O, IC2D.O, R10.2, R13.2, R16.2, R7.2
- net D1: now also IC2A.O, R7.2
- net D2: now also IC2B.O, R10.2
- net D3: now also IC2C.O, R13.2
- net D4: now also IC2D.O, R16.2
- net N$16: now also IC2E.I; no longer IC4F.I
- net N$22: now also IC2E.O; no longer IC4F.O
- net N$24: now also IC2F.I, IC3B.OUT; no longer IC4E.I, IC5A.OUT
- net N$25: now also IC3B.-IN; no longer IC5A.-IN
- net N$26: now also IC3B.+IN; no longer IC5A.+IN
- net N$30: now also IC2F.O; no longer IC4E.O
Other:
- moved on the sheet: IC2A, IC2B, IC2C, IC2D, LED2, LED3, LED4, LED5, R10, R11, R12, R13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
